Commit message: New features for Mapping

File: src/ballbot_description/urdf/ballbot.urdf.xacro (robot description, xacro)
@@ -143,3 +143,30 @@
     <axis xyz="0 0 0" />
   </joint>
+  <link name="laser_link">
+    <inertial>
+      <origin xyz="-0.011945780406062 -0.000381929217680526 -0.0170649378129477" rpy="0 0 0" />
+      <mass value="0.073084435549317" />
+      <inertia ixx="1.96074931730795E-05" ixy="-3.62091076640009E-07" ixz="4.28230084046735E-07"
+               iyy="2.40983835136327E-05" iyz="1.50180909250652E-08"
+               izz="4.14184164228595E-05" />
+    </inertial>
+    <visual>
+      <origin xyz="0.0 0.0 0.0" rpy="0 0 0" />
+      <geometry>
+          <mesh filename="package://ballbot_description/meshes/laser_link.STL"/>
+      </geometry>
+    </visual>
+    <collision>
+      <origin xyz="0.0 0.0 0.0" rpy="0 0 0" />
+      <geometry>
+          <mesh filename="package://ballbot_description/meshes/laser_link.STL" />
+      </geometry>
+    </collision>
+  </link>
+  <joint name="laser_joint" type="fixed">
+    <origin xyz="-0.0050526 -0.0023221 0.1208" rpy="0 0 3.14" />
+    <parent link="base_link" />
+    <child link="laser_link" />
+    <axis xyz="0 0 0" />
+  </joint>
 </robot>

File: src/ballbot_description/urdf/ballbot_gazebo.xacro (robot description, xacro)
@@ -41,4 +41,37 @@
     <parameters>$(find ballbot_controller)/config/ballbot_controllers.yaml</parameters>
   </plugin>
+  <plugin filename="gz-sim-imu-system" name="gz::sim::systems::Imu">
+  </plugin>
+  <plugin filename="gz-sim-sensors-system" name="gz::sim::systems::Sensors">
+    <render_engine>ogre2</render_engine>
+  </plugin>
+  </gazebo>
+ <gazebo reference="laser_link">
+    <sensor name="lidar" type="gpu_ray">
+      <always_on>true</always_on>
+      <update_rate>10</update_rate>
+      <visualize>true</visualize>
+      <topic>scan</topic>
+      <gz_frame_id>laser_link</gz_frame_id>
+      <ray>
+        <scan>
+          <horizontal>
+            <resolution>1.0</resolution>
+            <min_angle>0.0</min_angle>
+            <max_angle>6.28319</max_angle>
+          </horizontal>
+        </scan>
+        <range>
+          <min>0.12</min>
+          <max>12.0</max>
+          <resolution>0.02</resolution>
+        </range>
+        <noise>
+          <type>gaussian</type>
+          <mean>0.0</mean>
+          <stddev>0.01</stddev>
+        </noise>
+      </ray>
+    </sensor>
   </gazebo>
 </robot>

File: src/ballbot_description/urdf/ballbot_ros2_control.xacro (robot description, xacro)
@@ -4,4 +4,8 @@
         <hardware>
             <plugin>gz_ros2_control/GazeboSimSystem</plugin>
+        </hardware>
+        <hardware>
+            <plugin>bumperbot_firmware/BumperbotInterface</plugin>
+            <param name="port">/dev/ttyUSB0</param>
         </hardware>
         <joint name="wheel_right_joint">
@@ -22,8 +26,3 @@
         </joint>
     </ros2_control>
-    <gazebo>
-        <plugin filename="gz_ros2_control-system" name="gz_ros2_control::GazeboSimROS2ControlPlugin">
-            <parameters>$(find ballbot_controller)/config/ballbot_controllers.yaml</parameters>
-        </plugin>
-    </gazebo>
 </robot>
